File: hardware/panel.kicad_pcb (KiCad board)
At the start: 2 copper layers, 246.3 x 130.2 mm, 308 parts, among them J102 SENSOR, J401 USART, J601 RJ45, J602 RJ45, U201 MCP2551-I/SN, U202 MCP2515-xSO, U301 LM324, U401 ATMEGA328P-PU, U501 LM7805, Y201 16MHz, Y401 16MHz

Commit message: Scales added to  the panel and plotted.
Parts:
- removed the C102 at (247.0, 147.3)
- removed the C102 at (182.2, 147.3)
- removed the C102 at (117.5, 147.3)
- removed the C102 at (52.7, 147.3)
- removed the C201 at (253.3, 85.1)
- removed the C201 at (188.6, 85.1)
- removed the C201 at (123.8, 85.1)
- removed the C201 at (59.1, 85.1)
- removed the C202 at (245.7, 69.2)
- removed the C202 at (181.0, 69.2)
- removed the C202 at (116.2, 69.2)
- removed the C202 at (51.4, 69.2)
- removed the C203 at (260.9, 79.0)
- removed the C203 at (196.2, 79.0)
- removed the C203 at (131.4, 79.0)
- removed the C203 at (66.7, 79.0)
- removed the C204 at (258.8, 82.8)
- removed the C204 at (194.0, 82.8)
- removed the C204 at (129.3, 82.8)
- removed the C204 at (64.5, 82.8)
- removed the C205 at (250.5, 59.3)
- removed the C205 at (185.8, 59.3)
- removed the C205 at (121.0, 59.3)
- removed the C205 at (56.3, 59.3)
- removed the C301 at (238.5, 136.8)
- removed the C301 at (173.7, 136.8)
- removed the C301 at (109.0, 136.8)
- removed the C301 at (44.2, 136.8)
- removed the C302 at (245.1, 134.2)
- removed the C302 at (180.3, 134.2)
- removed the C302 at (115.6, 134.2)
- removed the C302 at (50.8, 134.2)
- removed the C303 at (249.3, 134.2)
- removed the C303 at (184.5, 134.2)
- removed the C303 at (119.8, 134.2)
- removed the C303 at (55.0, 134.2)
- removed the C304 at (241.0, 119.6)
- removed the C304 at (176.3, 119.6)
- removed the C304 at (111.5, 119.6)
- removed the C304 at (46.7, 119.6)
- removed the C401 at (242.3, 105.7)
- removed the C401 at (177.5, 105.7)
- removed the C401 at (112.8, 105.7)
- removed the C401 at (48.0, 105.7)
- removed the C402 at (257.5, 110.7)
- removed the C402 at (192.8, 110.7)
- removed the C402 at (128.0, 110.7)
- removed the C402 at (63.2, 110.7)
- removed the C403 at (260.1, 103.1)
- removed the C403 at (195.3, 103.1)
- removed the C403 at (130.5, 103.1)
- removed the C403 at (65.8, 103.1)
- removed the C404 at (258.8, 107.6)
- removed the C404 at (194.0, 107.6)
- removed the C404 at (129.3, 107.6)
- removed the C404 at (64.5, 107.6)
- removed the C405 at (258.8, 126.0)
- removed the C405 at (194.0, 126.0)
- removed the C405 at (129.3, 126.0)
- removed the C405 at (64.5, 126.0)
- removed the C406 at (255.4, 130.4)
- removed the C406 at (190.6, 130.4)
- removed the C406 at (125.8, 130.4)
- removed the C406 at (61.1, 130.4)
- removed the C501 at (230.3, 83.2)
- removed the C501 at (165.5, 83.2)
- removed the C501 at (100.7, 83.2)
- removed the C501 at (36.0, 83.2)
- removed the C502 at (230.2, 87.0)
- removed the C502 at (165.5, 87.0)
- removed the C502 at (100.7, 87.0)
- removed the C502 at (36.0, 87.0)
- removed the C503 at (236.8, 83.8)
- removed the C503 at (172.1, 83.8)
- removed the C503 at (107.3, 83.8)
- removed the C503 at (42.5, 83.8)
- removed the C504 at (236.8, 87.0)
- removed the C504 at (172.0, 87.0)
- removed the C504 at (107.3, 87.0)
- removed the C504 at (42.5, 87.0)
- removed the D101 at (258.8, 138.0)
- removed the D101 at (194.0, 138.0)
- removed the D101 at (129.3, 138.0)
- removed the D101 at (64.5, 138.0)
- removed the D201 at (242.2, 54.2)
- removed the D201 at (177.5, 54.2)
- removed the D201 at (112.7, 54.2)
- removed the D201 at (47.9, 54.2)
- removed the D301 at (238.7, 114.3)
- removed the D301 at (174.0, 114.3)
- removed the D301 at (109.2, 114.3)
- removed the D301 at (44.5, 114.3)
- removed the D401 at (258.8, 133.6)
- removed the D401 at (194.0, 133.6)
- removed the D401 at (129.3, 133.6)
- removed the D401 at (64.5, 133.6)
- removed the D402 at (263.9, 90.7)
- removed the D402 at (199.1, 90.7)
- removed the D402 at (134.4, 90.7)
- removed the D402 at (69.6, 90.7)
- removed the D403 at (263.9, 93.2)
- removed the D403 at (199.1, 93.2)
- removed the D403 at (134.4, 93.2)
- removed the D403 at (69.6, 93.2)
- removed the D501 at (224.8, 69.8)
- removed the D501 at (160.0, 69.8)
- removed the D501 at (95.2, 69.8)
- removed the D501 at (30.5, 69.8)
- removed the F501 at (224.8, 78.7)
- removed the F501 at (160.0, 78.7)
- removed the F501 at (95.2, 78.7)
- removed the F501 at (30.5, 78.7)
- removed the H101 at (266.4, 152.8)
- removed the H101 at (201.7, 152.8)
- removed the H101 at (136.9, 152.8)
- removed the H101 at (72.1, 152.8)
- removed the H102 at (266.4, 56.1)
- removed the H102 at (201.7, 56.1)
- removed the H102 at (136.9, 56.1)
- removed the H102 at (72.1, 56.1)
- removed the H103 at (223.2, 56.1)
- removed the H103 at (158.5, 56.1)
- removed the H103 at (93.7, 56.1)
- removed the H103 at (29.0, 56.1)
- removed the H104 at (223.2, 152.7)
- removed the H104 at (158.5, 152.7)
- removed the H104 at (93.7, 152.7)
- removed the H104 at (29.0, 152.7)
- removed the J102 at (249.5, 151.1)
- removed the J102 at (184.8, 151.1)
- removed the J102 at (120.0, 151.1)
- removed the J102 at (55.2, 151.1)
- removed the J401 at (266.4, 118.4)
- removed the J401 at (201.7, 118.4)
- removed the J401 at (136.9, 118.4)
- removed the J401 at (72.1, 118.4)
- removed the J601 at (239.7, 43.4)
- removed the J601 at (175.0, 43.4)
- removed the J601 at (110.2, 43.4)
- removed the J601 at (45.5, 43.4)
- removed the J602 at (260.6, 43.4)
- removed the J602 at (195.8, 43.4)
- removed the J602 at (131.1, 43.4)
- removed the J602 at (66.3, 43.4)
- removed the JP101 at (229.0, 152.4)
- removed the JP101 at (164.2, 152.4)
- removed the JP101 at (99.4, 152.4)
- removed the JP101 at (34.7, 152.4)
- removed the R201 at (242.2, 58.2)
- removed the R201 at (177.5, 58.2)
- removed the R201 at (112.7, 58.2)
- removed the R201 at (47.9, 58.2)
- removed the R202 at (250.5, 57.1)
- removed the R202 at (185.8, 57.1)
- removed the R202 at (121.0, 57.1)
- removed the R202 at (56.3, 57.1)
- removed the R203 at (242.3, 71.1)
- removed the R203 at (177.5, 71.1)
- removed the R203 at (112.8, 71.1)
- removed the R203 at (48.0, 71.1)
- removed the R301 at (234.0, 136.8)
- removed the R301 at (169.3, 136.8)
- removed the R301 at (104.5, 136.8)
- removed the R301 at (39.8, 136.8)
- removed the R302 at (228.3, 136.8)
- removed the R302 at (163.6, 136.8)
- removed the R302 at (98.8, 136.8)
- removed the R302 at (34.0, 136.8)
- removed the R303 at (232.5, 134.2)
- removed the R303 at (167.7, 134.2)
- removed the R303 at (103.0, 134.2)
- removed the R303 at (38.2, 134.2)
- removed the R304 at (228.3, 134.2)
- removed the R304 at (163.6, 134.2)
- removed the R304 at (98.8, 134.2)
- removed the R304 at (34.0, 134.2)
- removed the R305 at (236.7, 134.2)
- removed the R305 at (171.9, 134.2)
- removed the R305 at (107.2, 134.2)
- removed the R305 at (42.4, 134.2)
- removed the R306 at (240.9, 134.2)
- removed the R306 at (176.1, 134.2)
- removed the R306 at (111.4, 134.2)
- removed the R306 at (46.6, 134.2)
- removed the R307 at (242.9, 136.8)
- removed the R307 at (178.2, 136.8)
- removed the R307 at (113.4, 136.8)
- removed the R307 at (48.6, 136.8)
- removed the R308 at (230.9, 131.7)
- removed the R308 at (166.1, 131.7)
- removed the R308 at (101.3, 131.7)
- removed the R308 at (36.6, 131.7)
- removed the R309 at (230.9, 129.2)
- removed the R309 at (166.1, 129.2)
- removed the R309 at (101.3, 129.2)
- removed the R309 at (36.6, 129.2)
- removed the R401 at (258.8, 128.5)
- removed the R401 at (194.0, 128.5)
- removed the R401 at (129.3, 128.5)
- removed the R401 at (64.5, 128.5)
- removed the R402 at (258.8, 123.4)
- removed the R402 at (194.0, 123.4)
- removed the R402 at (129.3, 123.4)
- removed the R402 at (64.5, 123.4)
- removed the R403 at (258.8, 120.9)
- removed the R403 at (194.0, 120.9)
- removed the R403 at (129.3, 120.9)
- removed the R403 at (64.5, 120.9)
- removed the R404 at (260.1, 90.7)
- removed the R404 at (195.3, 90.7)
- removed the R404 at (130.5, 90.7)
- removed the R404 at (65.8, 90.7)
- removed the R405 at (260.1, 93.2)
- removed the R405 at (195.3, 93.2)
- removed the R405 at (130.5, 93.2)
- removed the R405 at (65.8, 93.2)
- removed the TP201 at (238.3, 77.5)
- removed the TP201 at (173.6, 77.5)
- removed the TP201 at (108.8, 77.5)
- removed the TP201 at (44.1, 77.5)
- removed the TP202 at (238.3, 74.3)
- removed the TP202 at (173.6, 74.3)
- removed the TP202 at (108.8, 74.3)
- removed the TP202 at (44.1, 74.3)
- removed the TP203 at (259.4, 66.9)
- removed the TP203 at (194.7, 66.9)
- removed the TP203 at (129.9, 66.9)
- removed the TP203 at (65.2, 66.9)
- removed the TP204 at (259.4, 70.7)
- removed the TP204 at (194.7, 70.7)
- removed the TP204 at (129.9, 70.7)
- removed the TP204 at (65.2, 70.7)
- removed the TP205 at (238.3, 71.1)
- removed the TP205 at (173.6, 71.1)
- removed the TP205 at (108.8, 71.1)
- removed the TP205 at (44.1, 71.1)
- removed the TP206 at (238.3, 80.6)
- removed the TP206 at (173.6, 80.6)
- removed the TP206 at (108.8, 80.6)
- removed the TP206 at (44.1, 80.6)
- removed the TP207 at (244.2, 61.0)
- removed the TP207 at (179.4, 61.0)
- removed the TP207 at (114.7, 61.0)
- removed the TP207 at (49.9, 61.0)
- removed the TP208 at (241.7, 64.4)
- removed the TP208 at (176.9, 64.4)
- removed the TP208 at (112.1, 64.4)
- removed the TP208 at (47.4, 64.4)
- removed the TP209 at (245.1, 89.9)
- removed the TP209 at (180.3, 89.9)
- removed the TP209 at (115.6, 89.9)
- removed the TP209 at (50.8, 89.9)
- removed the TP301 at (234.7, 141.2)
- removed the TP301 at (169.9, 141.2)
- removed the TP301 at (105.1, 141.2)
- removed the TP301 at (40.4, 141.2)
- removed the TP302 at (238.5, 141.2)
- removed the TP302 at (173.7, 141.2)
- removed the TP302 at (109.0, 141.2)
- removed the TP302 at (44.2, 141.2)
- removed the TP303 at (230.9, 141.2)
- removed the TP303 at (166.1, 141.2)
- removed the TP303 at (101.3, 141.2)
- removed the TP303 at (36.6, 141.2)
- removed the TP304 at (233.4, 119.6)
- removed the TP304 at (168.6, 119.6)
- removed the TP304 at (103.9, 119.6)
- removed the TP304 at (39.1, 119.6)
- removed the TP305 at (242.3, 141.2)
- removed the TP305 at (177.5, 141.2)
- removed the TP305 at (112.8, 141.2)
- removed the TP305 at (48.0, 141.2)
- removed the TP306 at (226.4, 131.1)
- removed the TP306 at (161.7, 131.1)
- removed the TP306 at (96.9, 131.1)
- removed the TP306 at (32.1, 131.1)
- removed the TP307 at (226.4, 127.3)
- removed the TP307 at (161.7, 127.3)
- removed the TP307 at (96.9, 127.3)
- removed the TP307 at (32.1, 127.3)
- removed the U201 at (250.5, 64.4)
- removed the U201 at (185.8, 64.4)
- removed the U201 at (121.0, 64.4)
- removed the U201 at (56.3, 64.4)
- removed the U202 at (250.5, 76.5)
- removed the U202 at (185.8, 76.5)
- removed the U202 at (121.0, 76.5)
- removed the U202 at (56.3, 76.5)
- removed the U301 at (238.5, 126.6)
- removed the U301 at (173.7, 126.6)
- removed the U301 at (109.0, 126.6)
- removed the U301 at (44.2, 126.6)
- removed the U401 at (253.7, 126.0)
- removed the U401 at (189.0, 126.0)
- removed the U401 at (124.2, 126.0)
- removed the U401 at (59.4, 126.0)
- removed the U501 at (231.1, 92.7)
- removed the U501 at (166.3, 92.7)
- removed the U501 at (101.6, 92.7)
- removed the U501 at (36.8, 92.7)
- removed the Y201 at (261.3, 76.5)
- removed the Y201 at (196.6, 76.5)
- removed the Y201 at (131.8, 76.5)
- removed the Y201 at (67.1, 76.5)
- removed the Y401 at (260.1, 100.6)
- removed the Y401 at (195.3, 100.6)
- removed the Y401 at (130.5, 100.6)
- removed the Y401 at (65.8, 100.6)
- added C102: 100nF, Capacitor_SMD:C_0805_2012Metric_Pad1.15x1.40mm_HandSolder, B.Cu at (247.0, 142.2)
- added C102: 100nF, Capacitor_SMD:C_0805_2012Metric_Pad1.15x1.40mm_HandSolder, B.Cu at (182.2, 142.2)
- added C102: 100nF, Capacitor_SMD:C_0805_2012Metric_Pad1.15x1.40mm_HandSolder, B.Cu at (117.5, 142.2)
- added C102: 100nF, Capacitor_SMD:C_0805_2012Metric_Pad1.15x1.40mm_HandSolder, B.Cu at (52.7, 142.2)
- added C201: 100nF, Capacitor_SMD:C_0805_2012Metric_Pad1.15x1.40mm_HandSolder, B.Cu at (253.3, 80.0)
- added C201: 100nF, Capacitor_SMD:C_0805_2012Metric_Pad1.15x1.40mm_HandSolder, B.Cu at (188.6, 80.0)
- added C201: 100nF, Capacitor_SMD:C_0805_2012Metric_Pad1.15x1.40mm_HandSolder, B.Cu at (123.8, 80.0)
- added C201: 100nF, Capacitor_SMD:C_0805_2012Metric_Pad1.15x1.40mm_HandSolder, B.Cu at (59.1, 80.0)
- added C202: 100nF, Capacitor_SMD:C_0805_2012Metric_Pad1.15x1.40mm_HandSolder, B.Cu at (245.7, 64.1)
- added C202: 100nF, Capacitor_SMD:C_0805_2012Metric_Pad1.15x1.40mm_HandSolder, B.Cu at (181.0, 64.1)
- added C202: 100nF, Capacitor_SMD:C_0805_2012Metric_Pad1.15x1.40mm_HandSolder, B.Cu at (116.2, 64.1)
- added C202: 100nF, Capacitor_SMD:C_0805_2012Metric_Pad1.15x1.40mm_HandSolder, B.Cu at (51.4, 64.1)
- added C203: 22pF, Capacitor_SMD:C_0805_2012Metric_Pad1.15x1.40mm_HandSolder, B.Cu at (260.9, 73.9)
- added C203: 22pF, Capacitor_SMD:C_0805_2012Metric_Pad1.15x1.40mm_HandSolder, B.Cu at (196.2, 73.9)
- added C203: 22pF, Capacitor_SMD:C_0805_2012Metric_Pad1.15x1.40mm_HandSolder, B.Cu at (131.4, 73.9)
- added C203: 22pF, Capacitor_SMD:C_0805_2012Metric_Pad1.15x1.40mm_HandSolder, B.Cu at (66.7, 73.9)
- added C204: 22pF, Capacitor_SMD:C_0805_2012Metric_Pad1.15x1.40mm_HandSolder, B.Cu at (258.8, 77.7)
- added C204: 22pF, Capacitor_SMD:C_0805_2012Metric_Pad1.15x1.40mm_HandSolder, B.Cu at (194.0, 77.7)
- added C204: 22pF, Capacitor_SMD:C_0805_2012Metric_Pad1.15x1.40mm_HandSolder, B.Cu at (129.3, 77.7)
- added C204: 22pF, Capacitor_SMD:C_0805_2012Metric_Pad1.15x1.40mm_HandSolder, B.Cu at (64.5, 77.7)
- added C205: 100nF, Capacitor_SMD:C_0805_2012Metric_Pad1.15x1.40mm_HandSolder, B.Cu at (250.5, 54.2)
- added C205: 100nF, Capacitor_SMD:C_0805_2012Metric_Pad1.15x1.40mm_HandSolder, B.Cu at (185.8, 54.2)
- added C205: 100nF, Capacitor_SMD:C_0805_2012Metric_Pad1.15x1.40mm_HandSolder, B.Cu at (121.0, 54.2)
- added C205: 100nF, Capacitor_SMD:C_0805_2012Metric_Pad1.15x1.40mm_HandSolder, B.Cu at (56.3, 54.2)
- added C301: 100n, Capacitor_SMD:C_0805_2012Metric_Pad1.15x1.40mm_HandSolder, B.Cu at (238.5, 131.7)
- added C301: 100n, Capacitor_SMD:C_0805_2012Metric_Pad1.15x1.40mm_HandSolder, B.Cu at (173.7, 131.7)
- added C301: 100n, Capacitor_SMD:C_0805_2012Metric_Pad1.15x1.40mm_HandSolder, B.Cu at (109.0, 131.7)
- added C301: 100n, Capacitor_SMD:C_0805_2012Metric_Pad1.15x1.40mm_HandSolder, B.Cu at (44.2, 131.7)
- added C302: 100n, Capacitor_SMD:C_0805_2012Metric_Pad1.15x1.40mm_HandSolder, B.Cu at (245.1, 129.2)
- added C302: 100n, Capacitor_SMD:C_0805_2012Metric_Pad1.15x1.40mm_HandSolder, B.Cu at (180.3, 129.2)
- added C302: 100n, Capacitor_SMD:C_0805_2012Metric_Pad1.15x1.40mm_HandSolder, B.Cu at (115.6, 129.2)
- added C302: 100n, Capacitor_SMD:C_0805_2012Metric_Pad1.15x1.40mm_HandSolder, B.Cu at (50.8, 129.2)
- added C303: 100n, Capacitor_SMD:C_0805_2012Metric_Pad1.15x1.40mm_HandSolder, B.Cu at (249.3, 129.2)
- added C303: 100n, Capacitor_SMD:C_0805_2012Metric_Pad1.15x1.40mm_HandSolder, B.Cu at (184.5, 129.2)
- added C303: 100n, Capacitor_SMD:C_0805_2012Metric_Pad1.15x1.40mm_HandSolder, B.Cu at (119.8, 129.2)
- added C303: 100n, Capacitor_SMD:C_0805_2012Metric_Pad1.15x1.40mm_HandSolder, B.Cu at (55.0, 129.2)
- added C304: 100n, Capacitor_SMD:C_0805_2012Metric_Pad1.15x1.40mm_HandSolder, B.Cu at (241.0, 114.6)
- added C304: 100n, Capacitor_SMD:C_0805_2012Metric_Pad1.15x1.40mm_HandSolder, B.Cu at (176.3, 114.6)
- added C304: 100n, Capacitor_SMD:C_0805_2012Metric_Pad1.15x1.40mm_HandSolder, B.Cu at (111.5, 114.6)
- added C304: 100n, Capacitor_SMD:C_0805_2012Metric_Pad1.15x1.40mm_HandSolder, B.Cu at (46.7, 114.6)
- added C401: 100nF, Capacitor_SMD:C_0805_2012Metric_Pad1.15x1.40mm_HandSolder, B.Cu at (242.3, 100.6)
- added C401: 100nF, Capacitor_SMD:C_0805_2012Metric_Pad1.15x1.40mm_HandSolder, B.Cu at (177.5, 100.6)
- added C401: 100nF, Capacitor_SMD:C_0805_2012Metric_Pad1.15x1.40mm_HandSolder, B.Cu at (112.8, 100.6)
- added C401: 100nF, Capacitor_SMD:C_0805_2012Metric_Pad1.15x1.40mm_HandSolder, B.Cu at (48.0, 100.6)
- added C402: 100nF, Capacitor_SMD:C_0805_2012Metric_Pad1.15x1.40mm_HandSolder, B.Cu at (257.5, 105.7)
- added C402: 100nF, Capacitor_SMD:C_0805_2012Metric_Pad1.15x1.40mm_HandSolder, B.Cu at (192.8, 105.7)
- added C402: 100nF, Capacitor_SMD:C_0805_2012Metric_Pad1.15x1.40mm_HandSolder, B.Cu at (128.0, 105.7)
- added C402: 100nF, Capacitor_SMD:C_0805_2012Metric_Pad1.15x1.40mm_HandSolder, B.Cu at (63.2, 105.7)
- added C403: 22pF, Capacitor_SMD:C_0805_2012Metric_Pad1.15x1.40mm_HandSolder, B.Cu at (260.1, 98.0)
- added C403: 22pF, Capacitor_SMD:C_0805_2012Metric_Pad1.15x1.40mm_HandSolder, B.Cu at (195.3, 98.0)
- added C403: 22pF, Capacitor_SMD:C_0805_2012Metric_Pad1.15x1.40mm_HandSolder, B.Cu at (130.5, 98.0)
- added C403: 22pF, Capacitor_SMD:C_0805_2012Metric_Pad1.15x1.40mm_HandSolder, B.Cu at (65.8, 98.0)
- added C404: 22pF, Capacitor_SMD:C_0805_2012Metric_Pad1.15x1.40mm_HandSolder, B.Cu at (258.8, 102.5)
- added C404: 22pF, Capacitor_SMD:C_0805_2012Metric_Pad1.15x1.40mm_HandSolder, B.Cu at (194.0, 102.5)
- added C404: 22pF, Capacitor_SMD:C_0805_2012Metric_Pad1.15x1.40mm_HandSolder, B.Cu at (129.3, 102.5)
- added C404: 22pF, Capacitor_SMD:C_0805_2012Metric_Pad1.15x1.40mm_HandSolder, B.Cu at (64.5, 102.5)
- added C405: 100nF, Capacitor_SMD:C_0805_2012Metric_Pad1.15x1.40mm_HandSolder, B.Cu at (258.8, 120.9)
- added C405: 100nF, Capacitor_SMD:C_0805_2012Metric_Pad1.15x1.40mm_HandSolder, B.Cu at (194.0, 120.9)
- added C405: 100nF, Capacitor_SMD:C_0805_2012Metric_Pad1.15x1.40mm_HandSolder, B.Cu at (129.3, 120.9)
- added C405: 100nF, Capacitor_SMD:C_0805_2012Metric_Pad1.15x1.40mm_HandSolder, B.Cu at (64.5, 120.9)
- added C406: 100nF, Capacitor_SMD:C_0805_2012Metric_Pad1.15x1.40mm_HandSolder, B.Cu at (255.4, 125.3)
- added C406: 100nF, Capacitor_SMD:C_0805_2012Metric_Pad1.15x1.40mm_HandSolder, B.Cu at (190.6, 125.3)
- added C406: 100nF, Capacitor_SMD:C_0805_2012Metric_Pad1.15x1.40mm_HandSolder, B.Cu at (125.8, 125.3)
- added C406: 100nF, Capacitor_SMD:C_0805_2012Metric_Pad1.15x1.40mm_HandSolder, B.Cu at (61.1, 125.3)
- added C501: 1uF, Capacitor_Tantalum_SMD:CP_EIA-6032-20_AVX-F_Pad2.25x2.35mm_HandSolder, B.Cu at (230.3, 78.1)
- added C501: 1uF, Capacitor_Tantalum_SMD:CP_EIA-6032-20_AVX-F_Pad2.25x2.35mm_HandSolder, B.Cu at (165.5, 78.1)
- added C501: 1uF, Capacitor_Tantalum_SMD:CP_EIA-6032-20_AVX-F_Pad2.25x2.35mm_HandSolder, B.Cu at (100.7, 78.1)
- added C501: 1uF, Capacitor_Tantalum_SMD:CP_EIA-6032-20_AVX-F_Pad2.25x2.35mm_HandSolder, B.Cu at (36.0, 78.1)
- added C502: 100nF, Capacitor_SMD:C_0805_2012Metric_Pad1.15x1.40mm_HandSolder, B.Cu at (230.2, 81.9)
- added C502: 100nF, Capacitor_SMD:C_0805_2012Metric_Pad1.15x1.40mm_HandSolder, B.Cu at (165.5, 81.9)
- added C502: 100nF, Capacitor_SMD:C_0805_2012Metric_Pad1.15x1.40mm_HandSolder, B.Cu at (100.7, 81.9)
- added C502: 100nF, Capacitor_SMD:C_0805_2012Metric_Pad1.15x1.40mm_HandSolder, B.Cu at (36.0, 81.9)
- added C503: 100nF, Capacitor_SMD:C_0805_2012Metric_Pad1.15x1.40mm_HandSolder, B.Cu at (236.8, 78.7)
- added C503: 100nF, Capacitor_SMD:C_0805_2012Metric_Pad1.15x1.40mm_HandSolder, B.Cu at (172.1, 78.7)
- added C503: 100nF, Capacitor_SMD:C_0805_2012Metric_Pad1.15x1.40mm_HandSolder, B.Cu at (107.3, 78.7)
- added C503: 100nF, Capacitor_SMD:C_0805_2012Metric_Pad1.15x1.40mm_HandSolder, B.Cu at (42.5, 78.7)
- added C504: 1uF, Capacitor_Tantalum_SMD:CP_EIA-6032-20_AVX-F_Pad2.25x2.35mm_HandSolder, B.Cu at (236.8, 81.9)
- added C504: 1uF, Capacitor_Tantalum_SMD:CP_EIA-6032-20_AVX-F_Pad2.25x2.35mm_HandSolder, B.Cu at (172.0, 81.9)
- added C504: 1uF, Capacitor_Tantalum_SMD:CP_EIA-6032-20_AVX-F_Pad2.25x2.35mm_HandSolder, B.Cu at (107.3, 81.9)
- added C504: 1uF, Capacitor_Tantalum_SMD:CP_EIA-6032-20_AVX-F_Pad2.25x2.35mm_HandSolder, B.Cu at (42.5, 81.9)
- added D101: LL4148, Diode_SMD:D_MiniMELF_Handsoldering, B.Cu at (258.8, 133.0)
- added D101: LL4148, Diode_SMD:D_MiniMELF_Handsoldering, B.Cu at (194.0, 133.0)
- added D101: LL4148, Diode_SMD:D_MiniMELF_Handsoldering, B.Cu at (129.3, 133.0)
- added D101: LL4148, Diode_SMD:D_MiniMELF_Handsoldering, B.Cu at (64.5, 133.0)
- added D201: pesd1can, Package_TO_SOT_SMD:SOT-23_Handsoldering, B.Cu at (242.2, 49.1)
- added D201: pesd1can, Package_TO_SOT_SMD:SOT-23_Handsoldering, B.Cu at (177.5, 49.1)
- added D201: pesd1can, Package_TO_SOT_SMD:SOT-23_Handsoldering, B.Cu at (112.7, 49.1)
- added D201: pesd1can, Package_TO_SOT_SMD:SOT-23_Handsoldering, B.Cu at (47.9, 49.1)
- added D301: 4V7, Diode_SMD:D_MiniMELF_Handsoldering, B.Cu at (238.7, 109.2)
- added D301: 4V7, Diode_SMD:D_MiniMELF_Handsoldering, B.Cu at (174.0, 109.2)
- added D301: 4V7, Diode_SMD:D_MiniMELF_Handsoldering, B.Cu at (109.2, 109.2)
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
Commit message: 7805 pad linked to GND, GND plane fixed below the sensor connector
Parts:
- removed the C102 at (247.0, 142.2)
- removed the C102 at (182.2, 142.2)
- removed the C102 at (117.5, 142.2)
- removed the C201 at (253.3, 80.0)
- removed the C201 at (188.6, 80.0)
- removed the C201 at (123.8, 80.0)
- removed the C202 at (245.7, 64.1)
- removed the C202 at (181.0, 64.1)
- removed the C202 at (116.2, 64.1)
- removed the C203 at (260.9, 73.9)
- removed the C203 at (196.2, 73.9)
- removed the C203 at (131.4, 73.9)
- removed the C204 at (258.8, 77.7)
- removed the C204 at (194.0, 77.7)
- removed the C204 at (129.3, 77.7)
- removed the C205 at (250.5, 54.2)
- removed the C205 at (185.8, 54.2)
- removed the C205 at (121.0, 54.2)
- removed the C301 at (238.5, 131.7)
- removed the C301 at (173.7, 131.7)
- removed the C301 at (109.0, 131.7)
- removed the C302 at (245.1, 129.2)
- removed the C302 at (180.3, 129.2)
- removed the C302 at (115.6, 129.2)
- removed the C303 at (249.3, 129.2)
- removed the C303 at (184.5, 129.2)
- removed the C303 at (119.8, 129.2)
- removed the C304 at (241.0, 114.6)
- removed the C304 at (176.3, 114.6)
- removed the C304 at (111.5, 114.6)
- removed the C401 at (242.3, 100.6)
- removed the C401 at (177.5, 100.6)
- removed the C401 at (112.8, 100.6)
- removed the C402 at (257.5, 105.7)
- removed the C402 at (192.8, 105.7)
- removed the C402 at (128.0, 105.7)
- removed the C403 at (260.1, 98.0)
- removed the C403 at (195.3, 98.0)
- removed the C403 at (130.5, 98.0)
- removed the C404 at (258.8, 102.5)
- removed the C404 at (194.0, 102.5)
- removed the C404 at (129.3, 102.5)
- removed the C405 at (258.8, 120.9)
- removed the C405 at (194.0, 120.9)
- removed the C405 at (129.3, 120.9)
- removed the C406 at (255.4, 125.3)
- removed the C406 at (190.6, 125.3)
- removed the C406 at (125.8, 125.3)
- removed the C501 at (230.3, 78.1)
- removed the C501 at (165.5, 78.1)
- removed the C501 at (100.7, 78.1)
- removed the C502 at (230.2, 81.9)
- removed the C502 at (165.5, 81.9)
- removed the C502 at (100.7, 81.9)
- removed the C503 at (236.8, 78.7)
- removed the C503 at (172.1, 78.7)
- removed the C503 at (107.3, 78.7)
- removed the C504 at (236.8, 81.9)
- removed the C504 at (172.0, 81.9)
- removed the C504 at (107.3, 81.9)
- removed the D101 at (258.8, 133.0)
- removed the D101 at (194.0, 133.0)
- removed the D101 at (129.3, 133.0)
- removed the D201 at (242.2, 49.1)
- removed the D201 at (177.5, 49.1)
- removed the D201 at (112.7, 49.1)
- removed the D301 at (238.7, 109.2)
- removed the D301 at (174.0, 109.2)
- removed the D301 at (109.2, 109.2)
- removed the D401 at (258.8, 128.5)
- removed the D401 at (194.0, 128.5)
- removed the D401 at (129.3, 128.5)
- removed the D402 at (263.9, 85.6)
- removed the D402 at (199.1, 85.6)
- removed the D402 at (134.4, 85.6)
- removed the D403 at (263.9, 88.2)
- removed the D403 at (199.1, 88.2)
- removed the D403 at (134.4, 88.2)
- removed the D501 at (224.8, 64.8)
- removed the D501 at (160.0, 64.8)
- removed the D501 at (95.2, 64.8)
- removed the F501 at (224.8, 73.7)
- removed the F501 at (160.0, 73.7)
- removed the F501 at (95.2, 73.7)
- removed the H101 at (266.4, 147.7)
- removed the H101 at (201.7, 147.7)
- removed the H101 at (136.9, 147.7)
- removed the H102 at (266.4, 51.1)
- removed the H102 at (201.7, 51.1)
- removed the H102 at (136.9, 51.1)
- removed the H103 at (223.2, 51.1)
- removed the H103 at (158.5, 51.1)
- removed the H103 at (93.7, 51.1)
- removed the H104 at (223.2, 147.6)
- removed the H104 at (158.5, 147.6)
- removed the H104 at (93.7, 147.6)
- removed the J102 at (249.5, 146.1)
- removed the J102 at (184.8, 146.1)
- removed the J102 at (120.0, 146.1)
- removed the J401 at (266.4, 113.3)
- removed the J401 at (201.7, 113.3)
- removed the J401 at (136.9, 113.3)
- removed the J601 at (239.7, 38.4)
- removed the J601 at (175.0, 38.4)
- removed the J601 at (110.2, 38.4)
- removed the J602 at (260.6, 38.4)
- removed the J602 at (195.8, 38.4)
- removed the J602 at (131.1, 38.4)
- removed the JP101 at (229.0, 147.3)
- removed the JP101 at (164.2, 147.3)
- removed the JP101 at (99.4, 147.3)
- removed the R201 at (242.2, 53.1)
- removed the R201 at (177.5, 53.1)
- removed the R201 at (112.7, 53.1)
- removed the R202 at (250.5, 52.1)
- removed the R202 at (185.8, 52.1)
- removed the R202 at (121.0, 52.1)
- removed the R203 at (242.3, 66.0)
- removed the R203 at (177.5, 66.0)
- removed the R203 at (112.8, 66.0)
- removed the R301 at (234.0, 131.7)
- removed the R301 at (169.3, 131.7)
- removed the R301 at (104.5, 131.7)
- removed the R302 at (228.3, 131.7)
- removed the R302 at (163.6, 131.7)
- removed the R302 at (98.8, 131.7)
- removed the R303 at (232.5, 129.2)
- removed the R303 at (167.7, 129.2)
- removed the R303 at (103.0, 129.2)
- removed the R304 at (228.3, 129.2)
- removed the R304 at (163.6, 129.2)
- removed the R304 at (98.8, 129.2)
- removed the R305 at (236.7, 129.2)
- removed the R305 at (171.9, 129.2)
- removed the R305 at (107.2, 129.2)
- removed the R306 at (240.9, 129.2)
- removed the R306 at (176.1, 129.2)
- removed the R306 at (111.4, 129.2)
- removed the R307 at (242.9, 131.7)
- removed the R307 at (178.2, 131.7)
- removed the R307 at (113.4, 131.7)
- removed the R308 at (230.9, 126.6)
- removed the R308 at (166.1, 126.6)
- removed the R308 at (101.3, 126.6)
- removed the R309 at (230.9, 124.1)
- removed the R309 at (166.1, 124.1)
- removed the R309 at (101.3, 124.1)
- removed the R401 at (258.8, 123.4)
- removed the R401 at (194.0, 123.4)
- removed the R401 at (129.3, 123.4)
- removed the R402 at (258.8, 118.4)
- removed the R402 at (194.0, 118.4)
- removed the R402 at (129.3, 118.4)
- removed the R403 at (258.8, 115.8)
- removed the R403 at (194.0, 115.8)
- removed the R403 at (129.3, 115.8)
- removed the R404 at (260.1, 85.6)
- removed the R404 at (195.3, 85.6)
- removed the R404 at (130.5, 85.6)
- removed the R405 at (260.1, 88.2)
- removed the R405 at (195.3, 88.2)
- removed the R405 at (130.5, 88.2)
- removed the TP201 at (238.3, 72.4)
- removed the TP201 at (173.6, 72.4)
- removed the TP201 at (108.8, 72.4)
- removed the TP202 at (238.3, 69.2)
- removed the TP202 at (173.6, 69.2)
- removed the TP202 at (108.8, 69.2)
- removed the TP203 at (259.4, 61.8)
- removed the TP203 at (194.7, 61.8)
- removed the TP203 at (129.9, 61.8)
- removed the TP204 at (259.4, 65.7)
- removed the TP204 at (194.7, 65.7)
- removed the TP204 at (129.9, 65.7)
- removed the TP205 at (238.3, 66.0)
- removed the TP205 at (173.6, 66.0)
- removed the TP205 at (108.8, 66.0)
- removed the TP206 at (238.3, 75.6)
- removed the TP206 at (173.6, 75.6)
- removed the TP206 at (108.8, 75.6)
- removed the TP207 at (244.2, 55.9)
- removed the TP207 at (179.4, 55.9)
- removed the TP207 at (114.7, 55.9)
- removed the TP208 at (241.7, 59.3)
- removed the TP208 at (176.9, 59.3)
- removed the TP208 at (112.1, 59.3)
- removed the TP209 at (245.1, 84.8)
- removed the TP209 at (180.3, 84.8)
- removed the TP209 at (115.6, 84.8)
- removed the TP301 at (234.7, 136.1)
- removed the TP301 at (169.9, 136.1)
- removed the TP301 at (105.1, 136.1)
- removed the TP302 at (238.5, 136.1)
- removed the TP302 at (173.7, 136.1)
- removed the TP302 at (109.0, 136.1)
- removed the TP303 at (230.9, 136.1)
- removed the TP303 at (166.1, 136.1)
- removed the TP303 at (101.3, 136.1)
- removed the TP304 at (233.4, 114.6)
- removed the TP304 at (168.6, 114.6)
- removed the TP304 at (103.9, 114.6)
- removed the TP305 at (242.3, 136.1)
- removed the TP305 at (177.5, 136.1)
- removed the TP305 at (112.8, 136.1)
- removed the TP306 at (226.4, 126.0)
- removed the TP306 at (161.7, 126.0)
- removed the TP306 at (96.9, 126.0)
- removed the TP307 at (226.4, 122.2)
- removed the TP307 at (161.7, 122.2)
- removed the TP307 at (96.9, 122.2)
- removed the U201 at (250.5, 59.3)
- removed the U201 at (185.8, 59.3)
- removed the U201 at (121.0, 59.3)
- removed the U202 at (250.5, 71.4)
- removed the U202 at (185.8, 71.4)
- removed the U202 at (121.0, 71.4)
- removed the U301 at (238.5, 121.5)
- removed the U301 at (173.7, 121.5)
- removed the U301 at (109.0, 121.5)
- removed the U401 at (253.7, 120.9)
- removed the U401 at (189.0, 120.9)
- removed the U401 at (124.2, 120.9)
- removed the U501 at (231.1, 87.6)
- removed the U501 at (166.3, 87.6)
- removed the U501 at (101.6, 87.6)
- removed the Y201 at (261.3, 71.4)
- removed the Y201 at (196.6, 71.4)
- removed the Y201 at (131.8, 71.4)
- removed the Y401 at (260.1, 95.5)
- removed the Y401 at (195.3, 95.5)
- removed the Y401 at (130.5, 95.5)
- added C102: 100nF, Capacitor_SMD:C_0805_2012Metric_Pad1.15x1.40mm_HandSolder, B.Cu at (240.3, 142.2)
- added C102: 100nF, Capacitor_SMD:C_0805_2012Metric_Pad1.15x1.40mm_HandSolder, B.Cu at (180.3, 142.2)
- added C102: 100nF, Capacitor_SMD:C_0805_2012Metric_Pad1.15x1.40mm_HandSolder, B.Cu at (120.3, 142.2)
- added C201: 100nF, Capacitor_SMD:C_0805_2012Metric_Pad1.15x1.40mm_HandSolder, B.Cu at (246.7, 80.0)
- added C201: 100nF, Capacitor_SMD:C_0805_2012Metric_Pad1.15x1.40mm_HandSolder, B.Cu at (186.7, 80.0)
- added C201: 100nF, Capacitor_SMD:C_0805_2012Metric_Pad1.15x1.40mm_HandSolder, B.Cu at (126.7, 80.0)
- added C202: 100nF, Capacitor_SMD:C_0805_2012Metric_Pad1.15x1.40mm_HandSolder, B.Cu at (239.1, 64.1)
- added C202: 100nF, Capacitor_SMD:C_0805_2012Metric_Pad1.15x1.40mm_HandSolder, B.Cu at (179.1, 64.1)
- added C202: 100nF, Capacitor_SMD:C_0805_2012Metric_Pad1.15x1.40mm_HandSolder, B.Cu at (119.1, 64.1)
- added C203: 22pF, Capacitor_SMD:C_0805_2012Metric_Pad1.15x1.40mm_HandSolder, B.Cu at (254.3, 73.9)
- added C203: 22pF, Capacitor_SMD:C_0805_2012Metric_Pad1.15x1.40mm_HandSolder, B.Cu at (194.3, 73.9)
- added C203: 22pF, Capacitor_SMD:C_0805_2012Metric_Pad1.15x1.40mm_HandSolder, B.Cu at (134.3, 73.9)
- added C204: 22pF, Capacitor_SMD:C_0805_2012Metric_Pad1.15x1.40mm_HandSolder, B.Cu at (252.1, 77.7)
- added C204: 22pF, Capacitor_SMD:C_0805_2012Metric_Pad1.15x1.40mm_HandSolder, B.Cu at (192.1, 77.7)
- added C204: 22pF, Capacitor_SMD:C_0805_2012Metric_Pad1.15x1.40mm_HandSolder, B.Cu at (132.1, 77.7)
- added C205: 100nF, Capacitor_SMD:C_0805_2012Metric_Pad1.15x1.40mm_HandSolder, B.Cu at (243.9, 54.2)
- added C205: 100nF, Capacitor_SMD:C_0805_2012Metric_Pad1.15x1.40mm_HandSolder, B.Cu at (183.9, 54.2)
- added C205: 100nF, Capacitor_SMD:C_0805_2012Metric_Pad1.15x1.40mm_HandSolder, B.Cu at (123.9, 54.2)
- added C301: 100n, Capacitor_SMD:C_0805_2012Metric_Pad1.15x1.40mm_HandSolder, B.Cu at (231.8, 131.7)
- added C301: 100n, Capacitor_SMD:C_0805_2012Metric_Pad1.15x1.40mm_HandSolder, B.Cu at (171.8, 131.7)
- added C301: 100n, Capacitor_SMD:C_0805_2012Metric_Pad1.15x1.40mm_HandSolder, B.Cu at (111.8, 131.7)
- added C302: 100n, Capacitor_SMD:C_0805_2012Metric_Pad1.15x1.40mm_HandSolder, B.Cu at (238.4, 129.2)
- added C302: 100n, Capacitor_SMD:C_0805_2012Metric_Pad1.15x1.40mm_HandSolder, B.Cu at (178.4, 129.2)
- added C302: 100n, Capacitor_SMD:C_0805_2012Metric_Pad1.15x1.40mm_HandSolder, B.Cu at (118.4, 129.2)
- added C303: 100n, Capacitor_SMD:C_0805_2012Metric_Pad1.15x1.40mm_HandSolder, B.Cu at (242.6, 129.2)
- added C303: 100n, Capacitor_SMD:C_0805_2012Metric_Pad1.15x1.40mm_HandSolder, B.Cu at (182.6, 129.2)
- added C303: 100n, Capacitor_SMD:C_0805_2012Metric_Pad1.15x1.40mm_HandSolder, B.Cu at (122.6, 129.2)
- added C304: 100n, Capacitor_SMD:C_0805_2012Metric_Pad1.15x1.40mm_HandSolder, B.Cu at (234.4, 114.6)
- added C304: 100n, Capacitor_SMD:C_0805_2012Metric_Pad1.15x1.40mm_HandSolder, B.Cu at (174.4, 114.6)
- added C304: 100n, Capacitor_SMD:C_0805_2012Metric_Pad1.15x1.40mm_HandSolder, B.Cu at (114.4, 114.6)
- added C401: 100nF, Capacitor_SMD:C_0805_2012Metric_Pad1.15x1.40mm_HandSolder, B.Cu at (235.6, 100.6)
- added C401: 100nF, Capacitor_SMD:C_0805_2012Metric_Pad1.15x1.40mm_HandSolder, B.Cu at (175.6, 100.6)
- added C401: 100nF, Capacitor_SMD:C_0805_2012Metric_Pad1.15x1.40mm_HandSolder, B.Cu at (115.6, 100.6)
- added C402: 100nF, Capacitor_SMD:C_0805_2012Metric_Pad1.15x1.40mm_HandSolder, B.Cu at (250.9, 105.7)
- added C402: 100nF, Capacitor_SMD:C_0805_2012Metric_Pad1.15x1.40mm_HandSolder, B.Cu at (190.9, 105.7)
- added C402: 100nF, Capacitor_SMD:C_0805_2012Metric_Pad1.15x1.40mm_HandSolder, B.Cu at (130.9, 105.7)
- added C403: 22pF, Capacitor_SMD:C_0805_2012Metric_Pad1.15x1.40mm_HandSolder, B.Cu at (253.4, 98.0)
- added C403: 22pF, Capacitor_SMD:C_0805_2012Metric_Pad1.15x1.40mm_HandSolder, B.Cu at (193.4, 98.0)
- added C403: 22pF, Capacitor_SMD:C_0805_2012Metric_Pad1.15x1.40mm_HandSolder, B.Cu at (133.4, 98.0)
- added C404: 22pF, Capacitor_SMD:C_0805_2012Metric_Pad1.15x1.40mm_HandSolder, B.Cu at (252.1, 102.5)
- added C404: 22pF, Capacitor_SMD:C_0805_2012Metric_Pad1.15x1.40mm_HandSolder, B.Cu at (192.1, 102.5)
- added C404: 22pF, Capacitor_SMD:C_0805_2012Metric_Pad1.15x1.40mm_HandSolder, B.Cu at (132.1, 102.5)
- added C405: 100nF, Capacitor_SMD:C_0805_2012Metric_Pad1.15x1.40mm_HandSolder, B.Cu at (252.1, 120.9)
- added C405: 100nF, Capacitor_SMD:C_0805_2012Metric_Pad1.15x1.40mm_HandSolder, B.Cu at (192.1, 120.9)
- added C405: 100nF, Capacitor_SMD:C_0805_2012Metric_Pad1.15x1.40mm_HandSolder, B.Cu at (132.1, 120.9)
- added C406: 100nF, Capacitor_SMD:C_0805_2012Metric_Pad1.15x1.40mm_HandSolder, B.Cu at (248.7, 125.3)
- added C406: 100nF, Capacitor_SMD:C_0805_2012Metric_Pad1.15x1.40mm_HandSolder, B.Cu at (188.7, 125.3)
- added C406: 100nF, Capacitor_SMD:C_0805_2012Metric_Pad1.15x1.40mm_HandSolder, B.Cu at (128.7, 125.3)
- added C501: 1uF, Capacitor_Tantalum_SMD:CP_EIA-6032-20_AVX-F_Pad2.25x2.35mm_HandSolder, B.Cu at (223.6, 78.1)
- added C501: 1uF, Capacitor_Tantalum_SMD:CP_EIA-6032-20_AVX-F_Pad2.25x2.35mm_HandSolder, B.Cu at (163.6, 78.1)
- added C501: 1uF, Capacitor_Tantalum_SMD:CP_EIA-6032-20_AVX-F_Pad2.25x2.35mm_HandSolder, B.Cu at (103.6, 78.1)
- added C502: 100nF, Capacitor_SMD:C_0805_2012Metric_Pad1.15x1.40mm_HandSolder, B.Cu at (223.6, 81.9)
- added C502: 100nF, Capacitor_SMD:C_0805_2012Metric_Pad1.15x1.40mm_HandSolder, B.Cu at (163.6, 81.9)
- added C502: 100nF, Capacitor_SMD:C_0805_2012Metric_Pad1.15x1.40mm_HandSolder, B.Cu at (103.6, 81.9)
- added C503: 100nF, Capacitor_SMD:C_0805_2012Metric_Pad1.15x1.40mm_HandSolder, B.Cu at (230.2, 78.7)
- added C503: 100nF, Capacitor_SMD:C_0805_2012Metric_Pad1.15x1.40mm_HandSolder, B.Cu at (170.2, 78.7)
- added C503: 100nF, Capacitor_SMD:C_0805_2012Metric_Pad1.15x1.40mm_HandSolder, B.Cu at (110.2, 78.7)
- added C504: 1uF, Capacitor_Tantalum_SMD:CP_EIA-6032-20_AVX-F_Pad2.25x2.35mm_HandSolder, B.Cu at (230.1, 81.9)
- added C504: 1uF, Capacitor_Tantalum_SMD:CP_EIA-6032-20_AVX-F_Pad2.25x2.35mm_HandSolder, B.Cu at (170.1, 81.9)
- added C504: 1uF, Capacitor_Tantalum_SMD:CP_EIA-6032-20_AVX-F_Pad2.25x2.35mm_HandSolder, B.Cu at (110.1, 81.9)
- added D101: LL4148, Diode_SMD:D_MiniMELF_Handsoldering, B.Cu at (252.1, 133.0)
- added D101: LL4148, Diode_SMD:D_MiniMELF_Handsoldering, B.Cu at (192.1, 133.0)
- added D101: LL4148, Diode_SMD:D_MiniMELF_Handsoldering, B.Cu at (132.1, 133.0)
- added D201: pesd1can, Package_TO_SOT_SMD:SOT-23_Handsoldering, B.Cu at (235.6, 49.1)
- added D201: pesd1can, Package_TO_SOT_SMD:SOT-23_Handsoldering, B.Cu at (175.6, 49.1)
- added D201: pesd1can, Package_TO_SOT_SMD:SOT-23_Handsoldering, B.Cu at (115.6, 49.1)
- added D301: 4V7, Diode_SMD:D_MiniMELF_Handsoldering, B.Cu at (232.1, 109.2)
- added D301: 4V7, Diode_SMD:D_MiniMELF_Handsoldering, B.Cu at (172.1, 109.2)
- added D301: 4V7, Diode_SMD:D_MiniMELF_Handsoldering, B.Cu at (112.1, 109.2)
- added D401: LL4148, Diode_SMD:D_MiniMELF_Handsoldering, B.Cu at (252.1, 128.5)
- added D401: LL4148, Diode_SMD:D_MiniMELF_Handsoldering, B.Cu at (192.1, 128.5)
- added D401: LL4148, Diode_SMD:D_MiniMELF_Handsoldering, B.Cu at (132.1, 128.5)
- added D402: LED_RED, LED_SMD:LED_0805_2012Metric_Pad1.15x1.40mm_HandSolder, B.Cu at (257.2, 85.6)
- added D402: LED_RED, LED_SMD:LED_0805_2012Metric_Pad1.15x1.40mm_HandSolder, B.Cu at (197.2, 85.6)
- added D402: LED_RED, LED_SMD:LED_0805_2012Metric_Pad1.15x1.40mm_HandSolder, B.Cu at (137.2, 85.6)
- added D403: LED_RED, LED_SMD:LED_0805_2012Metric_Pad1.15x1.40mm_HandSolder, B.Cu at (257.2, 88.2)
- added D403: LED_RED, LED_SMD:LED_0805_2012Metric_Pad1.15x1.40mm_HandSolder, B.Cu at (197.2, 88.2)
- added D403: LED_RED, LED_SMD:LED_0805_2012Metric_Pad1.15x1.40mm_HandSolder, B.Cu at (137.2, 88.2)
- added D501: LL4148, Diode_SMD:D_MiniMELF_Handsoldering, B.Cu at (218.1, 64.8)
- added D501: LL4148, Diode_SMD:D_MiniMELF_Handsoldering, B.Cu at (158.1, 64.8)
- added D501: LL4148, Diode_SMD:D_MiniMELF_Handsoldering, B.Cu at (98.1, 64.8)
- added F501: 500mA, Fuse:Fuse_1206_3216Metric_Pad1.42x1.75mm_HandSolder, B.Cu at (218.1, 73.7)
- added F501: 500mA, Fuse:Fuse_1206_3216Metric_Pad1.42x1.75mm_HandSolder, B.Cu at (158.1, 73.7)
- added F501: 500mA, Fuse:Fuse_1206_3216Metric_Pad1.42x1.75mm_HandSolder, B.Cu at (98.1, 73.7)
- added H101: MountingHole, MountingHole:MountingHole_3.2mm_M3, F.Cu at (259.8, 147.7)
- added H101: MountingHole, MountingHole:MountingHole_3.2mm_M3, F.Cu at (199.8, 147.7)
- added H101: MountingHole, MountingHole:MountingHole_3.2mm_M3, F.Cu at (139.8, 147.7)
- added H102: MountingHole, MountingHole:MountingHole_3.2mm_M3, F.Cu at (259.8, 51.1)
- added H102: MountingHole, MountingHole:MountingHole_3.2mm_M3, F.Cu at (199.8, 51.1)
- added H102: MountingHole, MountingHole:MountingHole_3.2mm_M3, F.Cu at (139.8, 51.1)
- added H103: MountingHole, MountingHole:MountingHole_3.2mm_M3, F.Cu at (216.6, 51.1)
- added H103: MountingHole, MountingHole:MountingHole_3.2mm_M3, F.Cu at (156.6, 51.1)
- added H103: MountingHole, MountingHole:MountingHole_3.2mm_M3, F.Cu at (96.6, 51.1)
- added H104: MountingHole, MountingHole:MountingHole_3.2mm_M3, F.Cu at (216.6, 147.6)
- added H104: MountingHole, MountingHole:MountingHole_3.2mm_M3, F.Cu at (156.6, 147.6)
- added H104: MountingHole, MountingHole:MountingHole_3.2mm_M3, F.Cu at (96.6, 147.6)
- added J102: SENSOR, TerminalBlock:TerminalBlock_bornier-4_P5.08mm, F.Cu at (242.9, 146.1)
- added J102: SENSOR, TerminalBlock:TerminalBlock_bornier-4_P5.08mm, F.Cu at (182.9, 146.1)
- added J102: SENSOR, TerminalBlock:TerminalBlock_bornier-4_P5.08mm, F.Cu at (122.9, 146.1)
- added J401: USART, Connector_PinHeader_2.54mm:PinHeader_1x04_P2.54mm_Vertical, F.Cu at (259.8, 113.3)
- added J401: USART, Connector_PinHeader_2.54mm:PinHeader_1x04_P2.54mm_Vertical, F.Cu at (199.8, 113.3)
- added J401: USART, Connector_PinHeader_2.54mm:PinHeader_1x04_P2.54mm_Vertical, F.Cu at (139.8, 113.3)
- added J601: RJ45, KicadZeniteSolarLibrary18:RJ45_YH59_01, F.Cu at (233.1, 38.4)
- added J601: RJ45, KicadZeniteSolarLibrary18:RJ45_YH59_01, F.Cu at (173.1, 38.4)
- added J601: RJ45, KicadZeniteSolarLibrary18:RJ45_YH59_01, F.Cu at (113.1, 38.4)
- added J602: RJ45, KicadZeniteSolarLibrary18:RJ45_YH59_01, F.Cu at (253.9, 38.4)
- added J602: RJ45, KicadZeniteSolarLibrary18:RJ45_YH59_01, F.Cu at (193.9, 38.4)
- added J602: RJ45, KicadZeniteSolarLibrary18:RJ45_YH59_01, F.Cu at (133.9, 38.4)
- added JP101: jmp, Jumper:SolderJumper-3_P1.3mm_Open_RoundedPad1.0x1.5mm, B.Cu at (222.3, 147.3)
- added JP101: jmp, Jumper:SolderJumper-3_P1.3mm_Open_RoundedPad1.0x1.5mm, B.Cu at (162.3, 147.3)
- added JP101: jmp, Jumper:SolderJumper-3_P1.3mm_Open_RoundedPad1.0x1.5mm, B.Cu at (102.3, 147.3)
- added R201: 120, Resistor_SMD:R_0805_2012Metric_Pad1.15x1.40mm_HandSolder, B.Cu at (235.6, 53.1)
- added R201: 120, Resistor_SMD:R_0805_2012Metric_Pad1.15x1.40mm_HandSolder, B.Cu at (175.6, 53.1)
- added R201: 120, Resistor_SMD:R_0805_2012Metric_Pad1.15x1.40mm_HandSolder, B.Cu at (115.6, 53.1)
- added R202: 4k7, Resistor_SMD:R_0805_2012Metric_Pad1.15x1.40mm_HandSolder, B.Cu at (243.9, 52.1)
- added R202: 4k7, Resistor_SMD:R_0805_2012Metric_Pad1.15x1.40mm_HandSolder, B.Cu at (183.9, 52.1)
- added R202: 4k7, Resistor_SMD:R_0805_2012Metric_Pad1.15x1.40mm_HandSolder, B.Cu at (123.9, 52.1)
- added R203: 10k, Resistor_SMD:R_0805_2012Metric_Pad1.15x1.40mm_HandSolder, B.Cu at (235.6, 66.0)
- added R203: 10k, Resistor_SMD:R_0805_2012Metric_Pad1.15x1.40mm_HandSolder, B.Cu at (175.6, 66.0)
- added R203: 10k, Resistor_SMD:R_0805_2012Metric_Pad1.15x1.40mm_HandSolder, B.Cu at (115.6, 66.0)
- added R301: 10k, Resistor_SMD:R_0805_2012Metric_Pad1.15x1.40mm_HandSolder, B.Cu at (227.4, 131.7)
- added R301: 10k, Resistor_SMD:R_0805_2012Metric_Pad1.15x1.40mm_HandSolder, B.Cu at (167.4, 131.7)
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Connections:
- U501 pad : (no net) -> GND
Other:
- board size 246.3 x 130.2 mm -> 232.1 x 131.2 mm
